File: business-card-pi-pico-pcb/business-card-pi-pico.kicad_sch (KiCad schematic)
At the start: 32 parts, among them U1 Pico

Commit message: continued working on PCB
continued working on PCB
Parts:
- added D31, D32, D33, D34, D35, D36: LED, LED_SMD:LED_0805_2012Metric, symbol Device:LED
- added R1, R2, R3, R4, R5, R6, R7: R, Resistor_SMD:R_0805_2012Metric, symbol Device:R
Connections:
- net at D10.2 (A), D11.2 (A), D13.1 (K)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: now also D25.2 (A), D26.1 (K), R6.2
- net at D11.1 (K), D13.2 (A), D17.2 (A)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: now also D27.2 (A), D28.1 (K), D29.2 (A), D30.1 (K), D31.2 (A), D32.1 (K), R7.2
- net pin1: now reaches U1.1 (GPIO0)
- net pin1: now also R1.1
- net pin2: now reaches U1.2 (GPIO1)
- net pin2: now also R2.1
- net pin3: now reaches U1.4 (GPIO2)
- net pin3: now also R3.1
- net pin4: now reaches U1.5 (GPIO3)
- net pin4: now also R4.1
- net pin5: now reaches U1.6 (GPIO4)
- net pin5: now also R5.1
- net pin6: now reaches U1.7 (GPIO5)
- net pin6: now also R6.1
- net pin7: now reaches U1.9 (GPIO6)
- net pin7: now also R7.1
- net at D10.1 (K), D15.2 (A), D16.1 (K)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: now also D19.2 (A), D20.1 (K), D35.2 (A), D36.1 (K), R5.2
- net at D12.2 (A), D14.1 (K), D15.1 (K)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: now also D27.1 (K), D28.2 (A), R3.2
- net at D1.2 (A), D12.1 (K), D14.2 (A)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: now also D19.1 (K), D20.2 (A), D25.1 (K), D26.2 (A), D31.1 (K), D32.2 (A), R1.2
- net at D1.1 (K), D2.2 (A), D3.2 (A)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: now also D29.1 (K), D30.2 (A), D33.1 (K), D34.2 (A), D35.1 (K), D36.2 (A), R2.2
- net at D17.1 (K), D18.2 (A), D23.2 (A)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: now also D33.2 (A), D34.1 (K), R4.2
Other:
- moved on the sheet: BT1, D1, D10, D11, D12, D13, D14, D15, D16, D17, D18, D19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
