File: business-card-pi-pico-pcb/_autosave-business-card-pi-pico.kicad_sch (KiCad schematic)
At the start: 44 parts, among them U1 Pico

Commit message: PCB updated a bit
PCB updated a bit
Other:
- moved on the sheet: D1, D10, D11, D12, D13, D14, D15, D16, D17, D18, D19, D2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
